File: SMD-Temperature-Controller/Temperature-Controller/Temperature-Controller.kicad_pcb (KiCad board)
At the start: 2 copper layers, 7 parts, among them J1 Screw_Terminal_01x02, J2 Screw_Terminal_01x02, J3 Screw_Terminal_01x02, J4 Screw_Terminal_01x03, J5 Screw_Terminal_01x03, J6 Screw_Terminal_01x03, U2 ESP32-S3

Commit message: Ready for creating the Gerber files
Parts:
- removed U2: ESP32-S3, Package_DFN_QFN:QFN-56-1EP_7x7mm_P0.4mm_EP4x4mm
- added C1: 0.1µF, ESP32_Custom_Footprints:C_Disc_D3.0mm_W1.6mm_P2.50mm, F.Cu at (124.5, 80.0)
- added C2: 1000µF C_Polarized, Capacitor_SMD:CP_Elec_8x10.5, F.Cu at (130.9, 87.6)
- added C3: 0.1µF, ESP32_Custom_Footprints:C_Disc_D3.0mm_W1.6mm_P2.50mm, F.Cu at (113.0, 86.3)
- added H1: MountingHole, ESP32_Custom_Footprints:MountingHole_3.2mm_M3_ISO7380, F.Cu at (33.0, 25.8)
- added H2: MountingHole, ESP32_Custom_Footprints:MountingHole_3.2mm_M3_ISO7380, F.Cu at (33.0, 33.0)
- added H3: MountingHole, ESP32_Custom_Footprints:MountingHole_3.2mm_M3_ISO7380, F.Cu at (33.0, 40.3)
- added H4: MountingHole, ESP32_Custom_Footprints:MountingHole_3.2mm_M3_ISO7380, F.Cu at (33.0, 47.5)
- added R1: 300Ω, Resistor_SMD:R_0805_2012Metric, F.Cu at (116.8, 62.6)
- added R2: 220Ω, Resistor_SMD:R_0805_2012Metric, F.Cu at (150.8, 82.5)
- added R3: 10KΩ, Resistor_SMD:R_0805_2012Metric, F.Cu at (121.9, 85.4)
- added R4: 10KΩ, Resistor_SMD:R_0805_2012Metric, F.Cu at (116.8, 85.4)
- added R5: 4.7KΩ, Resistor_SMD:R_0805_2012Metric, F.Cu at (116.8, 71.5)
- added R6: 220Ω, Resistor_SMD:R_0805_2012Metric, F.Cu at (116.8, 81.6)
- added U1: ESP32-S3-MINI-1U, RF_Module:ESP32-S2-MINI-1U, F.Cu at (134.0, 73.0)
- J1: value Screw_Terminal_01x02 -> RGB_LED Terminal; footprint TerminalBlock:TerminalBlock_MaiXu_MX126-5.0-02P_1x02_P5.00mm -> ESP32_Custom_Footprints:TerminalBlock_bornier-3_P5.08mm
- J2: value Screw_Terminal_01x02 -> DS18B20 Terminal; footprint TerminalBlock:TerminalBlock_MaiXu_MX126-5.0-02P_1x02_P5.00mm -> ESP32_Custom_Footprints:TerminalBlock_bornier-3_P5.08mm
- J3: value Screw_Terminal_01x02 -> SSR_25DA_Terminal; footprint TerminalBlock:TerminalBlock_MaiXu_MX126-5.0-02P_1x02_P5.00mm -> TerminalBlock_4Ucon:TerminalBlock_4Ucon_1x02_P3.50mm_Horizontal
- J4: value Screw_Terminal_01x03 -> Power Input Terminal; footprint ESP32_Custom_Footprints:TerminalBlock_bornier-3_P5.08mm -> TerminalBlock_4Ucon:TerminalBlock_4Ucon_1x02_P3.50mm_Horizontal
- J5: value Screw_Terminal_01x03 -> SCT 013-020 Terminal; footprint ESP32_Custom_Footprints:TerminalBlock_bornier-3_P5.08mm -> TerminalBlock_4Ucon:TerminalBlock_4Ucon_1x02_P3.50mm_Horizontal
- J6: value Screw_Terminal_01x03 -> Red LED Power Indicator; footprint ESP32_Custom_Footprints:TerminalBlock_bornier-3_P5.08mm -> TerminalBlock_4Ucon:TerminalBlock_4Ucon_1x02_P3.50mm_Horizontal
- moved J6 135.6 mm to (149.9, 74.0), turned to -90 degrees
- moved J1 126.7 mm to (128.3, 57.1)
- moved J5 105.9 mm to (105.4, 84.1), turned to -90 degrees
- moved J3 104.8 mm to (105.4, 74.9), turned to -90 degrees
- moved J2 102.2 mm to (105.4, 58.4), turned to -90 degrees
- moved J4 87.5 mm to (146.1, 88.9), turned to 180 degrees
Connections:
- J1 pad 1: unconnected-(J1-Pin_1-Pad1) -> GND
- J1 pad 2: unconnected-(J1-Pin_2-Pad2) -> Net-(J1-Pin_2)
- J2 pad 1: unconnected-(J2-Pin_1-Pad1) -> GND
- J2 pad 2: unconnected-(J2-Pin_2-Pad2) -> /GPIO25
- J3 pad 1: unconnected-(J3-Pin_1-Pad1) -> GND
- J3 pad 2: unconnected-(J3-Pin_2-Pad2) -> /GPIO26
- J4 pad 1: unconnected-(J4-Pin_1-Pad1) -> GND
- J4 pad 2: unconnected-(J4-Pin_2-Pad2) -> +5V
- J5 pad 1: unconnected-(J5-Pin_1-Pad1) -> GND
- J5 pad 2: unconnected-(J5-Pin_2-Pad2) -> Net-(J5-Pin_2)
- J6 pad 1: unconnected-(J6-Pin_1-Pad1) -> GND
- J6 pad 2: unconnected-(J6-Pin_2-Pad2) -> Net-(J6-Pin_2)
Routing:
- net /GPIO25: track 0.00 -> 25.5 mm
- net /GPIO26: track 0.00 -> 23.5 mm
- net +3.3V: track 0.00 -> 22.7 mm
- net Net-(J1-Pin_2): track 0.00 -> 18.4 mm
- net /GPIO27: track 0.00 -> 13.7 mm
- net Net-(C3-Pad2): track 0.00 -> 11.2 mm
- net Net-(J5-Pin_2): track 0.00 -> 8.16 mm
- net Net-(J6-Pin_2): track 0.00 -> 5.08 mm
- added copper zone on F.Cu, net +5V
- added copper zone on B.Cu, net GND
Other:
- board outline added: 65 x 50 mm
- board text added: "0.1µF"
