File: SMD-Temperature-Controller/Temperature-Controller/Temperature-Controller.kicad_sch (KiCad schematic)
At the start: 7 parts, among them J1 Screw_Terminal_01x02, J2 Screw_Terminal_01x02, J3 Screw_Terminal_01x02, J4 Screw_Terminal_01x03, J5 Screw_Terminal_01x03, J6 Screw_Terminal_01x03, U2 ESP32-S3

Commit message: Ready for creating the Gerber files
Parts:
- removed J1, J2: Screw_Terminal_01x02, TerminalBlock:TerminalBlock_MaiXu_MX126-5.0-02P_1x02_P5.00mm, symbol ESP32-Custom-Symbols:Screw_Terminal_01x02
- removed J4, J5: Screw_Terminal_01x03, ESP32_Custom_Footprints:TerminalBlock_bornier-3_P5.08mm, symbol ESP32-Custom-Symbols:Screw_Terminal_01x03
- removed U2: ESP32-S3, Package_DFN_QFN:QFN-56-1EP_7x7mm_P0.4mm_EP4x4mm, symbol MCU_Espressif:ESP32-S3
- added C1, C3: 0.1µF Ceramic Capacitor, ESP32_Custom_Footprints:C_Disc_D3.0mm_W1.6mm_P2.50mm, symbol ESP32-Custom-Symbols:0.1µF_Ceramic_Capacitor
- added C2: 1000µF C_Polarized, Capacitor_SMD:CP_Elec_8x10.5, symbol ESP32-Custom-Symbols:C_Polarized
- added H1, H2, H3, H4: MountingHole, ESP32_Custom_Footprints:MountingHole_3.2mm_M3_ISO7380, symbol Mechanical:MountingHole
- added J2: DS18B20 Terminal, ESP32_Custom_Footprints:TerminalBlock_bornier-3_P5.08mm, symbol ESP32-Custom-Symbols:Screw_Terminal_01x03
- added J4: Power Input Terminal, TerminalBlock_4Ucon:TerminalBlock_4Ucon_1x02_P3.50mm_Horizontal, symbol ESP32-Custom-Symbols:Screw_Terminal_01x02
- added J5: SCT 013-020 Terminal, TerminalBlock_4Ucon:TerminalBlock_4Ucon_1x02_P3.50mm_Horizontal, symbol ESP32-Custom-Symbols:Screw_Terminal_01x02
- added J6: Red LED Power Indicator, TerminalBlock_4Ucon:TerminalBlock_4Ucon_1x02_P3.50mm_Horizontal, symbol ESP32-Custom-Symbols:Screw_Terminal_01x02
- added R1: 300Ω, Resistor_SMD:R_0805_2012Metric, symbol Device:R
- added R2, R6: 220Ω, Resistor_SMD:R_0805_2012Metric, symbol Device:R
- added R3, R4: 10KΩ, Resistor_SMD:R_0805_2012Metric, symbol Device:R
- added R5: 4.7KΩ, Resistor_SMD:R_0805_2012Metric, symbol Device:R
- added U1: ESP32-S3-MINI-1U, RF_Module:ESP32-S2-MINI-1U, symbol ESP32-Custom-Symbols:ESP32-S3-MINI-1U
- J1: renamed from J6; value Screw_Terminal_01x03 -> RGB_LED Terminal
- J3: value Screw_Terminal_01x02 -> SSR_25DA_Terminal; footprint TerminalBlock:TerminalBlock_MaiXu_MX126-5.0-02P_1x02_P5.00mm -> TerminalBlock_4Ucon:TerminalBlock_4Ucon_1x02_P3.50mm_Horizontal
Connections:
- net GND: now reaches J3.1 (Pin_1)
- net GND: now also J1.1 (Pin_1), C1.1, C2.1, J2.1 (Pin_1), J4.1 (Pin_1), J5.1 (Pin_1), J6.1 (Pin_1), R4.1, U1.14 (GND1), U1.29 (GND)
- net GPIO26: now reaches J3.2 (Pin_2)
- net GPIO26: now also U1.9 (GPIO26)
- net at J1.2 (Pin_2): now also R1.1
- net +5V: now reaches J1.3 (Pin_3)
- net +5V: now also C1.2, C2.2, J2.3 (Pin_3), J4.2 (Pin_2), R2.2, R5.2, U1.15 (+5V)
- new net: C3.1, J5.2 (Pin_2)
- new net: C3.2, R3.1, R4.2, R6.1
- new net: J6.2 (Pin_2), R2.1
- new net +3.3V: R3.2, U1.30 (3V3)
- new net GPIO233: R1.2
- new net GPIO25: J2.2 (Pin_2), R5.1, U1.8 (GPIO25)
- new net GPIO27: R6.2, U1.10 (GPIO27)
- new net GPIO33: U1.7 (GPIO33)
- no-connect marks 0 -> 22
Other:
- note added: "DS18B20 +5V"
- note added: "DS18B20 Data"
- note added: "DS18B20 GND"
- note added: "LED +5V"
- note added: "LED GND"
- note added: "LED ON/OFF"
- note added: "Power Input GND"
- note added: "Power input +5V"
- note added: "RED LED +5v"
- note added: "RED LED GND"
- note added: "RSS_25 Open/Closed"
- note added: "RSS_25DA GND"
- note added: "SCT 013020 Current Detetion"
- note added: "SCT 013020 GND"
- moved on the sheet: J1
