File: Temperature-Controller/Temperature-Controller.kicad_pcb (KiCad board)
At the start: 2 copper layers, 66 x 98.4 mm, 20 parts, among them J1 RGB LED Terminal, J2 DS18B20 Terminal, J3 SSR_25DA Terminal, J4 Power Input Terminal, J5 SCT-013-020 Current Sensor Te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, J6 Red LED Power Indecator

Commit message: Ready for creating the Gerber files
Parts:
- removed C5: 0.1µF Ceramic Capacitor, ESP32_Custom_Footprints:C_Disc_D3.0mm_W1.6mm_P2.50mm
- J5: value SCT-013-020 Current Sensor Terminal -> SCT 013 020 Indecator; footprint ESP32_Custom_Footprints:TerminalBlock_bornier-3_P5.08mm -> ESP32_Custom_Footprints:TerminalBlock_bornier-2_P5.08mm
- moved C3 11.3 mm to (203.2, 116.8)
- moved R5 6.29 mm to (213.4, 111.8)
- moved R4 5.14 mm to (196.8, 111.8)
- moved J5 2.03 mm to (195.6, 124.5)
Connections:
- C3 pad 1: GND -> Net-(J5-Pin_2)
- J5 pad 2: /GPIO33 -> Net-(J5-Pin_2)
Routing:
- net +3.3V: track 35.5 -> 18.8 mm
- net /GPIO33: track 67.5 -> 53.1 mm
- net Net-(J5-Pin_2): track 0.00 -> 8.67 mm
